File: HW4/HW4_KiCad/HW4_KiCad.kicad_sch (KiCad schematic)
At the start: 23 parts, among them J1 Header, 6 Pin, J2 Header, 2 Pin, J3 Header, 12 Pin, J4 Header, 12 Pin, SW1 Button, SW2 Button, SW3 Slide Switch, U1 AP7381, U2 PIC32MX170F256B

Commit message: hw4 update
Other:
- note added: "2 inch square board Remember the capacitors that are supposed to be close to the PIC Careful not to orphan grounds"
Changed lines of the file:
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@@
     (stroke (width 0) (type default) (color 0 0 0 0))
+  )
+  (text "2 inch square board\nRemember the capacitors that are supposed to be close to the PIC\nCareful not to orphan grounds\n"
+    (at 39.37 151.13 0)
+    (effects (font (size 1.27 1.27)) (justify left bottom))
   )
   (global_label "V_{IN}" (shape passive) (at 207.01 127 0) (fields_autoplaced)

Commit message: update hw4, add readme
Parts:
- C1, C2, C3, C4, C5, C6: footprint (none) -> ME_433:Capacitor
- D1, D2, D3: footprint (none) -> ME_433:LED
- J1: footprint (none) -> ME_433:CP2102 Header
- J2: footprint (none) -> ME_433:Battery Connector
- J3, J4: footprint (none) -> ME_433:Side Header
- R1, R2, R3, R4, R5: footprint (none) -> ME_433:Resistor
- SW1, SW2: footprint (none) -> ME_433:Button
- SW3: footprint (none) -> ME_433:Switch
- U1: footprint (none) -> ME_433:AP7381
- U2: footprint (none) -> ME_433:PIC Socket
Connections:
- net V_{IN}: now also C2.1, SW3.2 (B), U1.3 (V_{IN})
